Commit message: Data from cameras, imu, gps, lidar fetched as well as teleop done

File: src/rover_description/urdf/rover.urdf (robot description, URDF)
Before this commit: robot mars_rover, 16 links, 15 joints
Links:
- added link lidar_link, mass 0.1; collision cylinder length=0.04 radius=0.05; visual cylinder length=0.04 radius=0.05
Joints:
- added joint lidar_joint: type fixed, parent chassis, child lidar_link, origin xyz=0 0 0.2 rpy=0 0 0

Commit message: map building started

File: src/rover_description/urdf/rover.urdf (robot description, URDF)
Before this commit: robot mars_rover, 17 links, 16 joints
Joints:
- removed joint base_footprint_tf
- added joint base_footprint_joint: type fixed, parent base_footprint, child base_link, origin xyz=0 0 0 rpy=0 0 0

Commit message: started nav but facing issue in map frame

File: src/rover_description/urdf/rover.urdf (robot description, URDF)
Before this commit: robot mars_rover, 17 links, 16 joints
Joints:
- joint wheel_1: limit (none) -> effort=100.0 velocity=20.0
- joint wheel_2: limit (none) -> effort=100.0 velocity=20.0
- joint wheel_3: limit (none) -> effort=100.0 velocity=20.0
- joint wheel_4: limit (none) -> effort=100.0 velocity=20.0

Commit message: updated navigation package

File: src/rover_description/urdf/rover.urdf (robot description, URDF)
Before this commit: robot mars_rover, 17 links, 16 joints
Links:
- link steering1: mass 6.64830273269256 -> 0.5
- link steering2: mass 6.64830400801289 -> 0.5
- link steering3: mass 6.64830392215954 -> 0.5
- link steering4: mass 6.64830259385427 -> 0.5
Joints:
- joint wheel_1: limit effort=100.0 velocity=20.0 -> effort=1000.0 velocity=20.0
- joint wheel_2: limit effort=100.0 velocity=20.0 -> effort=1000.0 velocity=20.0
- joint wheel_3: limit effort=100.0 velocity=20.0 -> effort=1000.0 velocity=20.0
- joint wheel_4: limit effort=100.0 velocity=20.0 -> effort=1000.0 velocity=20.0

Commit message: fixes

File: src/rover_description/urdf/rover.urdf (robot description, URDF)
Before this commit: robot mars_rover, 17 links, 16 joints
Joints:
- removed joint wheel_1
- removed joint wheel_2
- removed joint wheel_3
- removed joint wheel_4
- added joint front_left_wheel_joint: type continuous, parent steering1, child wheel1, origin xyz=0.000353156675627797 0.0676257237290513 -0.216586122585117 rpy=-1.5708332999603 1.83526331234849E-05 0.00321478961806723, axis 0 0 1, limit effort=1000.0 velocity=20.0
- added joint front_right_wheel_joint: type continuous, parent steering2, child wheel2, origin xyz=0.00260503655999339 -0.0673405250297557 -0.216999105202697 rpy=-1.5707963267949 0 0.0261401718711602, axis 0 0 1, limit effort=1000.0 velocity=20.0
- added joint rear_left_wheel_joint: type continuous, parent steering4, child wheel4, origin xyz=-0.00146559562126541 0.0673855594536285 -0.21697972522299 rpy=-1.5707963246485 1.83519361346148E-05 0.00917303616199558, axis 0 0 1, limit effort=1000.0 velocity=20.0
- added joint rear_right_wheel_joint: type continuous, parent steering3, child wheel3, origin xyz=-0.000555418729084156 -0.067625619393596 -0.216581022537134 rpy=-1.5707963267949 0 0, axis 0 0 1, limit effort=1000.0 velocity=20.0

Commit message: saving code

File: src/rover_description/urdf/rover.urdf (robot description, URDF)
Before this commit: robot mars_rover, 17 links, 16 joints
Joints:
- removed joint wheel_1
- removed joint wheel_2
- removed joint wheel_3
- removed joint wheel_4
- added joint front_left_wheel_joint: type continuous, parent steering1, child wheel1, origin xyz=0.000353156675627797 0.0676257237290513 -0.216586122585117 rpy=-1.5708332999603 1.83526331234849E-05 0.00321478961806723, axis 0 0 1, limit effort=1000.0 velocity=20.0
- added joint front_right_wheel_joint: type continuous, parent steering4, child wheel4, origin xyz=-0.00146559562126541 0.0673855594536285 -0.21697972522299 rpy=-1.5707963246485 1.83519361346148E-05 0.00917303616199558, axis 0 0 1, limit effort=1000.0 velocity=20.0
- added joint rear_left_wheel_joint: type continuous, parent steering2, child wheel2, origin xyz=0.00260503655999339 -0.0673405250297557 -0.216999105202697 rpy=-1.5707963267949 0 0.0261401718711602, axis 0 0 1, limit effort=1000.0 velocity=20.0
- added joint rear_right_wheel_joint: type continuous, parent steering3, child wheel3, origin xyz=-0.000555418729084156 -0.067625619393596 -0.216581022537134 rpy=-1.5707963267949 0 0, axis 0 0 1, limit effort=1000.0 velocity=20.0
